File: inducter_tx.kicad_pcb (KiCad board)
At the start: 2 copper layers, 79 x 134 mm, 18 parts, among them J1 Jack-DC, Q1 NMOS, Q2 NMOS, U1 4047, U2 TC4426xOA

Commit message: Add files via upload
updated design
Parts:
- moved C7 31.2 mm to (122.1, 159.1), turned to 180 degrees
- moved U2 27.2 mm to (124.4, 145.2)
- moved C6 12.7 mm to (118.0, 146.9), turned to 0 degrees
- moved C2 12.3 mm to (112.6, 148.7), turned to 180 degrees
- moved C4 10.3 mm to (81.2, 145.2), turned to 180 degrees
- moved R3 9.82 mm to (112.1, 142.6), turned to 180 degrees
- moved R1 9.54 mm to (112.6, 150.7), turned to 180 degrees
- moved C1 6.75 mm to (82.7, 136.6)
- moved Q1 5.59 mm to (91.7, 140.5)
- moved C5 4.81 mm to (111.8, 157.0)
- moved R2 4.79 mm to (96.5, 144.8), turned to 180 degrees
- moved Q2 3.75 mm to (104.3, 140.5), turned to 180 degrees
- moved U1 3.60 mm to (118.2, 153.3), turned to 0 degrees
- moved C3 3.01 mm to (81.5, 150.8), turned to 180 degrees
Routing:
- net Net-(U2-~{OUT_A}): track 4.70 -> 28.0 mm, vias 0 -> 2
- net Net-(U2-~{OUT_B}): track 4.09 -> 17.9 mm, vias 0 -> 2
- net GND: track 51.5 -> 41.0 mm, vias 14 -> 13
- net Net-(C1-Pad1): track 17.4 -> 7.51 mm
- net Net-(Q1-S): track 26.3 -> 16.9 mm
- net Net-(U1-Q): track 17.9 -> 8.84 mm
- net Net-(U1-~{Q}): track 16.7 -> 8.63 mm
- net +12V: track 86.5 -> 84.9 mm, vias 2 -> 3
- net Net-(Q1-G): track 3.43 -> 2.46 mm
- net Net-(Q2-G): track 2.04 -> 2.73 mm
- removed copper zone on F.Cu, net +12V
