File: inducter_tx.kicad_sch (KiCad schematic)
At the start: 18 parts, among them J1 Jack-DC, Q1 NMOS, Q2 NMOS, U1 4047, U2 TC4426xOA

Commit message: Add files via upload
updated design
Other:
- title: (none) -> inducter_tx
Changed lines of the file:
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@@
 	(generator_version "9.0")
 	(paper "A4")
+	(title_block
+		(title "inducter_tx")
+		(date "2026-03-12")
+		(rev "ver 2.0")
+	)
 	(junction
 		(at 21.59 87.63)
@@
 	(wire
 		(pts
-			(xy 137.16 45.72) (xy 137.16 100.33)
+			(xy 137.16 45.72) (xy 137.16 46.99)
 		)
 		(stroke
@@
 	(wire
 		(pts
-			(xy 101.6 45.72) (xy 101.6 100.33)
-		)
-		(stroke
-			(width 0)
-			(type default)
-		)
-	)
-	(wire
-		(pts
-			(xy 73.66 45.72) (xy 73.66 101.6)
+			(xy 101.6 45.72) (xy 101.6 46.99)
+		)
+		(stroke
+			(width 0)
+			(type default)
+		)
+	)
+	(wire
+		(pts
+			(xy 73.66 45.72) (xy 73.66 46.99)
 		)
 		(stroke
@@
 	(wire
 		(pts
-			(xy 59.69 34.29) (xy 59.69 38.1)
+			(xy 59.69 33.02) (xy 59.69 38.1)
 		)
 		(stroke
@@
 	(wire
 		(pts
-			(xy 17.78 99.06) (xy 17.78 101.6)
+			(xy 19.05 99.06) (xy 19.05 101.6)
 		)
 		(stroke
@@
 	(wire
 		(pts
-			(xy 127 45.72) (xy 127 100.33)
+			(xy 127 45.72) (xy 127 46.99)
 		)
 		(stroke
@@
 	(wire
 		(pts
-			(xy 19.05 99.06) (xy 17.78 99.06)
-		)
-		(stroke
-			(width 0)
-			(type default)
-		)
-	)
-	(wire
-		(pts
-			(xy 80.01 45.72) (xy 80.01 101.6)
+			(xy 80.01 45.72) (xy 80.01 46.99)
 		)
 		(stroke
@@
 	(symbol
 		(lib_id "power:GND")
-		(at 137.16 100.33 0)
+		(at 137.16 46.99 0)
 		(unit 1)
 		(exclude_from_sim no)
@@
 		(fields_autoplaced yes)
 		(property "Reference" "#PWR012"
-			(at 137.16 106.68 0)
+			(at 137.16 53.34 0)
 			(effects
 				(font
@@
 		)
 		(property "Value" "GND"
-			(at 137.16 105.41 0)
+			(at 137.16 52.07 0)
 			(effects
 				(font
@@
 		)
 		(property "Footprint" ""
-			(at 137.16 100.33 0)
+			(at 137.16 46.99 0)
 			(effects
 				(font
@@
 		)
 		(property "Datasheet" ""
-			(at 137.16 100.33 0)
+			(at 137.16 46.99 0)
 			(effects
 				(font
@@
 		)
 		(property "Description" "Power symbol creates a global label with name \"GND\" , ground"
-			(at 137.16 100.33 0)
+			(at 137.16 46.99 0)
 			(effects
 				(font
@@
 	(symbol
 		(lib_id "power:GND")
-		(at 73.66 101.6 0)
+		(at 73.66 46.99 0)
 		(unit 1)
 		(exclude_from_sim no)
@@
 		(fields_autoplaced yes)
 		(property "Reference" "#PWR015"
-			(at 73.66 107.95 0)
+			(at 73.66 53.34 0)
 			(effects
 				(font
@@
 		)
 		(property "Value" "GND"
-			(at 73.66 106.68 0)
+			(at 73.66 52.07 0)
 			(effects
 				(font
@@
 		)
 		(property "Footprint" ""
-			(at 73.66 101.6 0)
+			(at 73.66 46.99 0)
 			(effects
 				(font
@@
 		)
 		(property "Datasheet" ""
-			(at 73.66 101.6 0)
+			(at 73.66 46.99 0)
 			(effects
 				(font
@@
 		)
 		(property "Description" "Power symbol creates a global label with name \"GND\" , ground"
-			(at 73.66 101.6 0)
+			(at 73.66 46.99 0)
 			(effects
 				(font
@@
 	(symbol
 		(lib_id "power:GND")
-		(at 17.78 101.6 0)
+		(at 19.05 101.6 0)
 		(unit 1)
 		(exclude_from_sim no)
@@
 		(fields_autoplaced yes)
 		(property "Reference" "#PWR016"
-			(at 17.78 107.95 0)
+			(at 19.05 107.95 0)
 			(effects
 				(font
@@
 		)
 		(property "Value" "GND"
-			(at 17.78 106.68 0)
+			(at 19.05 106.68 0)
 			(effects
 				(font
@@
 		)
 		(property "Footprint" ""
-			(at 17.78 101.6 0)
+			(at 19.05 101.6 0)
 			(effects
 				(font
@@
 		)
 		(property "Datasheet" ""
-			(at 17.78 101.6 0)
+			(at 19.05 101.6 0)
 			(effects
 				(font
@@
 		)
 		(property "Description" "Power symbol creates a global label with name \"GND\" , ground"
-			(at 17.78 101.6 0)
+			(at 19.05 101.6 0)
 			(effects
 				(font
@@
 	(symbol
 		(lib_id "power:GND")
-		(at 127 100.33 0)
+		(at 127 46.99 0)
 		(unit 1)
 		(exclude_from_sim no)
@@
 		(fields_autoplaced yes)
 		(property "Reference" "#PWR011"
-			(at 127 106.68 0)
+			(at 127 53.34 0)
 			(effects
 				(font
@@
 		)
 		(property "Value" "GND"
-			(at 127 105.41 0)
+			(at 127 52.07 0)
 			(effects
 				(font
@@
 		)
 		(property "Footprint" ""
-			(at 127 100.33 0)
+			(at 127 46.99 0)
 			(effects
 				(font
@@
 		)
 		(property "Datasheet" ""
-			(at 127 100.33 0)
+			(at 127 46.99 0)
 			(effects
 				(font
@@
 		)
 		(property "Description" "Power symbol creates a global label with name \"GND\" , ground"
-			(at 127 100.33 0)
+			(at 127 46.99 0)
 			(effects
 				(font
@@
 	(symbol
 		(lib_id "power:GND")
-		(at 80.01 101.6 0)
+		(at 80.01 46.99 0)
 		(unit 1)
 		(exclude_from_sim no)
@@
 		(fields_autoplaced yes)
 		(property "Reference" "#PWR017"
-			(at 80.01 107.95 0)
+			(at 80.01 53.34 0)
 			(effects
 				(font
@@
 		)
 		(property "Value" "GND"
-			(at 80.01 106.68 0)
+			(at 80.01 52.07 0)
 			(effects
 				(font
@@
 		)
 		(property "Footprint" ""
-			(at 80.01 101.6 0)
+			(at 80.01 46.99 0)
 			(effects
 				(font
@@
 		)
 		(property "Datasheet" ""
-			(at 80.01 101.6 0)
+			(at 80.01 46.99 0)
 			(effects
 				(font
@@
 		)
 		(property "Description" "Power symbol creates a global label with name \"GND\" , ground"
-			(at 80.01 101.6 0)
+			(at 80.01 46.99 0)
 			(effects
 				(font
@@
 	(symbol
 		(lib_id "power:+12V")
-		(at 59.69 34.29 0)
+		(at 59.69 33.02 0)
 		(unit 1)
 		(exclude_from_sim no)
@@
 		(fields_autoplaced yes)
 		(property "Reference" "#PWR01"
-			(at 59.69 38.1 0)
+			(at 59.69 36.83 0)
 			(effects
 				(font
@@
 		)
 		(property "Value" "+12V"
-			(at 59.69 29.21 0)
+			(at 59.69 27.94 0)
 			(effects
 				(font
@@
 		)
 		(property "Footprint" ""
-			(at 59.69 34.29 0)
+			(at 59.69 33.02 0)
 			(effects
 				(font
@@
 		)
 		(property "Datasheet" ""
-			(at 59.69 34.29 0)
+			(at 59.69 33.02 0)
 			(effects
 				(font
@@
 		)
 		(property "Description" "Power symbol creates a global label with name \"+12V\""
-			(at 59.69 34.29 0)
+			(at 59.69 33.02 0)
 			(effects
 				(font
@@
 	(symbol
 		(lib_id "power:GND")
-		(at 101.6 100.33 0)
+		(at 101.6 46.99 0)
 		(unit 1)
 		(exclude_from_sim no)
@@
 		(fields_autoplaced yes)
 		(property "Reference" "#PWR018"
-			(at 101.6 106.68 0)
+			(at 101.6 53.34 0)
 			(effects
 				(font
@@
 		)
 		(property "Value" "GND"
-			(at 101.6 105.41 0)
+			(at 101.6 52.07 0)
 			(effects
 				(font
@@
 		)
 		(property "Footprint" ""
-			(at 101.6 100.33 0)
+			(at 101.6 46.99 0)
 			(effects
 				(font
@@
 		)
 		(property "Datasheet" ""
-			(at 101.6 100.33 0)
+			(at 101.6 46.99 0)
 			(effects
 				(font
@@
 		)
 		(property "Description" "Power symbol creates a global label with name \"GND\" , ground"
-			(at 101.6 100.33 0)
-			(effects
-				(font
+			(at 101.6 46.99 0)
+			(effects
+				(font
